Commit message: fanuc and motoman in xacro displayed in rviz

File: nistfanuc_ws/src/fanuc_lrmate200id_support/urdf/lrmate200id (copy).xacro (robot description, xacro)
@@ -3,9 +3,6 @@
   <xacro:include filename="$(find fanuc_lrmate200id_support)/urdf/lrmate200id_macro.xacro"/>
    <xacro:include filename="$(find fanuc_lrmate200id_support)/urdf/robotiq_c2_model_macro.xacro"/>
-   <xacro:include filename="$(find motoman_sia20d_support)/urdf/sia20d_macro.xacro"/>
     <xacro:fanuc_lrmate200id prefix="fanuc_"/>
    <xacro:robotiq_c2_model prefix="fanuc_"/>
-    <xacro:motoman_sia20d prefix="motoman_"/>
-   <xacro:robotiq_c2_model prefix="motoman_"/>
   <link name="world" />
   <!-- Dummy Link -->
@@ -19,5 +16,5 @@
   <!--[ERROR] [1474736838.974400369]: joint 'fanuc_joint_6-tool0' is not unique.-->
   <!-- First Robot -->
-  <joint name="fanuc_joint_0" type="fixed">
+  <joint name="joint_0" type="fixed">
     <parent link="link0" />
     <child link="fanuc_base_link" />
@@ -31,15 +28,3 @@
     <axis xyz="0 0 0"/>
   </joint>
-  <!-- Second Robot -->
-  <joint name="motoman_joint_0" type="fixed">
-    <parent link="link0" />
-    <child link="motoman_base_link" />
-    <origin xyz="0 0.5 0" rpy="0 0 0"/>
-  </joint>
-   <joint name="motoman_link_t-tool0" type="fixed" >
-     <!--  <origin xyz="0 0 0.0" rpy="0 0 -3.1416"/> -->
-     <origin xyz="0 0 0.0" rpy="0  -1.57  0"/>
-      <parent link="motoman_link_t" />
-      <child link="motoman_robotiq_85_adapter_link" />
-     </joint>
 </robot>
