Commit message: two robot checkers

File: checkers_ws/src/fanuc_lrmate200id_support/urdf/lrmate200id.urdf (robot description, URDF)
Before this commit: robot fanuc_lrmate200id, 9 links, 8 joints
Links:
- removed link base
- removed link tool0
- added link link0
- added link robotiq_85_adapter_link; collision mesh filename=package://fanuc_lrmate200id_support/meshes/robotiq_c2/colli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; visual mesh filename=package://fanuc_lrmate200id_support/meshes/robotiq_c2/visua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
- added link robotiq_85_base_link; collision mesh filename=package://fanuc_lrmate200id_support/meshes/robotiq_c2/colli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; visual mesh filename=package://fanuc_lrmate200id_support/meshes/robotiq_c2/visua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
- added link robotiq_85_left_finger_link; collision mesh filename=package://fanuc_lrmate200id_support/meshes/robotiq_c2/colli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; visual mesh filename=package://fanuc_lrmate200id_support/meshes/robotiq_c2/visua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
- added link robotiq_85_left_finger_tip_link; collision mesh filename=package://fanuc_lrmate200id_support/meshes/robotiq_c2/colli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; visual mesh filename=package://fanuc_lrmate200id_support/meshes/robotiq_c2/visua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
- added link robotiq_85_left_inner_knuckle_link; collision mesh filename=package://fanuc_lrmate200id_support/meshes/robotiq_c2/colli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; visual mesh filename=package://fanuc_lrmate200id_support/meshes/robotiq_c2/visua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
- added link robotiq_85_left_knuckle_link; collision mesh filename=package://fanuc_lrmate200id_support/meshes/robotiq_c2/colli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; visual mesh filename=package://fanuc_lrmate200id_support/meshes/robotiq_c2/visua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
- added link robotiq_85_right_finger_link; collision mesh filename=package://fanuc_lrmate200id_support/meshes/robotiq_c2/colli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; visual mesh filename=package://fanuc_lrmate200id_support/meshes/robotiq_c2/visua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
- added link robotiq_85_right_finger_tip_link; collision mesh filename=package://fanuc_lrmate200id_support/meshes/robotiq_c2/colli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; visual mesh filename=package://fanuc_lrmate200id_support/meshes/robotiq_c2/visua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
- added link robotiq_85_right_inner_knuckle_link; collision mesh filename=package://fanuc_lrmate200id_support/meshes/robotiq_c2/colli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; visual mesh filename=package://fanuc_lrmate200id_support/meshes/robotiq_c2/visua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
- added link robotiq_85_right_knuckle_link; collision mesh filename=package://fanuc_lrmate200id_support/meshes/robotiq_c2/colli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; visual mesh filename=package://fanuc_lrmate200id_support/meshes/robotiq_c2/visua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
- added link world
- link base_link: geometry collision mesh filename=package://fanuc_lrmate200id_support/meshes/lrmate200id/visu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 scale=1.0 1.0 1.0; visual mesh filename=package://fanuc_lrmate200id_support/meshes/lrmate200id/visu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 scale=1.0 1.0 1.0
- link link_1: geometry collision mesh filename=package://fanuc_lrmate200id_support/meshes/lrmate200id/visu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 scale=1.0 1.0 1.0; visual mesh filename=package://fanuc_lrmate200id_support/meshes/lrmate200id/visu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 scale=1.0 1.0 1.0
- link link_2: geometry collision mesh filename=package://fanuc_lrmate200id_support/meshes/lrmate200id/visu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 scale=1.0 1.0 1.0; visual mesh filename=package://fanuc_lrmate200id_support/meshes/lrmate200id/visu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 scale=1.0 1.0 1.0
- link link_3: geometry collision mesh filename=package://fanuc_lrmate200id_support/meshes/lrmate200id/visu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 scale=1.0 1.0 1.0; visual mesh filename=package://fanuc_lrmate200id_support/meshes/lrmate200id/visu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 scale=1.0 1.0 1.0
- link link_4: geometry collision mesh filename=package://fanuc_lrmate200id_support/meshes/lrmate200id/visu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 scale=1.0 1.0 1.0; visual mesh filename=package://fanuc_lrmate200id_support/meshes/lrmate200id/visu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 scale=1.0 1.0 1.0
- link link_5: geometry collision mesh filename=package://fanuc_lrmate200id_support/meshes/lrmate200id/visu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 scale=1.0 1.0 1.0; visual mesh filename=package://fanuc_lrmate200id_support/meshes/lrmate200id/visu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 scale=1.0 1.0 1.0
- link link_6: geometry collision mesh filename=package://fanuc_lrmate200id_support/meshes/lrmate200id/visu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 scale=1.0 1.0 1.0; visual mesh filename=package://fanuc_lrmate200id_support/meshes/lrmate200id/visu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 scale=1.0 1.0 1.0
Joints:
- removed joint base_link-base
- added joint joint_0: type fixed, parent link0, child base_link, origin xyz=0 -0.5 0 rpy=0 0 0
- added joint robotiq_85_base_joint: type fixed, parent robotiq_85_adapter_link, child robotiq_85_base_link, origin xyz=.0085 0 -.0041 rpy=0 0 0, axis 1 0 0
- added joint robotiq_85_left_finger_joint: type fixed, parent robotiq_85_left_knuckle_link, child robotiq_85_left_finger_link, origin xyz=0 .00508 .03134 rpy=3.1415 0 0, axis 1 0 0, limit lower=0 upper=1.5707 effort=1000 velocity=2.0
- added joint robotiq_85_left_finger_tip_joint: type revolute, parent robotiq_85_left_inner_knuckle_link, child robotiq_85_left_finger_tip_link, origin xyz=0 .04196 -.0388 rpy=0 0 0, axis 1 0 0, limit lower=0 upper=1.5707 effort=1000 velocity=2.0, mimic joint=robotiq_85_left_knuckle_joint multiplier=-1
- added joint robotiq_85_left_inner_knuckle_joint: type revolute, parent robotiq_85_base_link, child robotiq_85_left_inner_knuckle_link, origin xyz=.04843 .0127 0 rpy=1.5707 1.5707 0, axis 1 0 0, limit lower=0 upper=1.5707 effort=1000 velocity=2.0, mimic joint=robotiq_85_left_knuckle_joint offset=0
- added joint robotiq_85_left_knuckle_joint: type revolute, parent robotiq_85_base_link, child robotiq_85_left_knuckle_link, origin xyz=.04191 .0306 0 rpy=-1.5707 1.5707 0, axis 1 0 0, limit lower=0 upper=.8575 effort=1000 velocity=2.0
- added joint robotiq_85_right_finger_joint: type fixed, parent robotiq_85_right_knuckle_link, child robotiq_85_right_finger_link, origin xyz=0 .00508 .03134 rpy=3.1415 0 0, axis 1 0 0, limit lower=0 upper=1.5707 effort=1000 velocity=2.0
- added joint robotiq_85_right_finger_tip_joint: type revolute, parent robotiq_85_right_inner_knuckle_link, child robotiq_85_right_finger_tip_link, origin xyz=0 .04196 -.0388 rpy=0 0 0, axis 1 0 0, limit lower=0 upper=1.5707 effort=1000 velocity=2.0, mimic joint=robotiq_85_left_knuckle_joint multiplier=-1
- added joint robotiq_85_right_inner_knuckle_joint: type revolute, parent robotiq_85_base_link, child robotiq_85_right_inner_knuckle_link, origin xyz=.04843 -.0127 0 rpy=-1.5707 -1.5707 0, axis 1 0 0, limit lower=0 upper=1.5707 effort=1000 velocity=2.0, mimic joint=robotiq_85_left_knuckle_joint offset=0
- added joint robotiq_85_right_knuckle_joint: type revolute, parent robotiq_85_base_link, child robotiq_85_right_knuckle_link, origin xyz=.04191 -.0306 0 rpy=1.5707 -1.5707 0, axis 1 0 0, limit lower=0 upper=1.5707 effort=1000 velocity=2.0, mimic joint=robotiq_85_left_knuckle_joint multiplier=1
- added joint world_joint: type fixed, parent world, child link0, origin xyz=0 0 0 rpy=0 0 0, axis 0 0 1
- joint joint_1: origin xyz=0 0 0.330 rpy=0 0 0 -> xyz=0 -0.5 0.330 rpy=0 0 0
- joint joint_4: limit lower=-3.315 upper=3.315 effort=0 velocity=9.60 -> lower=-3.315 upper=3.315 effort=0 velocity=9.6
- joint joint_6: axis 1 0 0 -> -1 0 0
- joint joint_6-tool0: axis 1 0 0 -> 0 0 0; child tool0 -> robotiq_85_adapter_link; origin xyz=0.0 0 0.0 rpy=3.1415926535 -1.570796327 0 -> xyz=0 0 0 rpy=0 0 0

File: checkers_ws/src/fanuc_lrmate200id_support/urdf/lrmate200id.xacro (robot description, xacro)
@@ -2,4 +2,44 @@
 <robot name="fanuc_lrmate200id" xmlns:xacro="http://ros.org/wiki/xacro">
   <xacro:include filename="$(find fanuc_lrmate200id_support)/urdf/lrmate200id_macro.xacro"/>
-  <xacro:fanuc_lrmate200id prefix=""/>
+   <xacro:include filename="$(find fanuc_lrmate200id_support)/urdf/robotiq_c2_model_macro.xacro"/>
+   <xacro:include filename="$(find motoman_sia20d_support)/urdf/sia20d_macro.xacro"/>
+    <xacro:fanuc_lrmate200id prefix="fanuc_"/>
+   <xacro:robotiq_c2_model prefix="fanuc_"/>
+    <xacro:motoman_sia20d prefix="motoman_"/>
+   <xacro:robotiq_c2_model prefix="motoman_"/>
+  <link name="world" />
+  <!-- Dummy Link -->
+  <link name="link0" />
+  <joint name="world_joint" type="fixed">
+    <parent link="world" />
+    <child link="link0" />
+    <origin xyz="0 0 0" rpy="0 0 0"/>
+    <axis xyz="0 0 1"/>
+  </joint>
+  <!--[ERROR] [1474736838.974400369]: joint 'fanuc_joint_6-tool0' is not unique.-->
+  <!-- First Robot -->
+  <joint name="fanuc_joint_0" type="fixed">
+    <parent link="link0" />
+    <child link="fanuc_base_link" />
+    <origin xyz="0 -0.5 0" rpy="0 0 0"/>
+  </joint>
+  <joint name="fanuc_joint_6-tool0" type="fixed">
+    <!--      <origin xyz="0 0 0" rpy="${m_pi} ${-m_pi_2} 0" /> -->
+    <origin xyz="0 0 0" rpy="0 0 0" />
+    <parent link="fanuc_link_6" />
+    <child link="fanuc_robotiq_85_adapter_link" />
+    <axis xyz="0 0 0"/>
+  </joint>
+  <!-- Second Robot -->
+  <joint name="motoman_joint_0" type="fixed">
+    <parent link="link0" />
+    <child link="motoman_base_link" />
+    <origin xyz="0 0.5 0" rpy="0 0 0"/>
+  </joint>
+   <joint name="motoman_link_t-tool0" type="fixed" >
+     <!--  <origin xyz="0 0 0.0" rpy="0 0 -3.1416"/> -->
+     <origin xyz="0 0 0.0" rpy="0  -1.57  0"/>
+      <parent link="motoman_link_t" />
+      <child link="motoman_robotiq_85_adapter_link" />
+     </joint>
 </robot>

File: checkers_ws/src/fanuc_lrmate200id_support/urdf/lrmate200id_macro.xacro (robot description, xacro)
@@ -9,5 +9,5 @@
     <link name="${prefix}base_link">
       <visual>
-        <origin xyz="0 0 0" rpy="0 0 0"/>
+        <origin rpy="0 0 0" xyz="0 0 0"/>
 	<xacro:insert_mesh_base_link />
         <xacro:material_fanuc_gray28 />
@@ -127,11 +127,4 @@
       <limit effort="${joint6effort}" lower="${joint6lower}" upper="${joint6upper}" velocity="${joint6velocity}" />
     </joint>
-    <joint name="${prefix}joint_6-tool0" type="fixed">
-<!--      <origin xyz="0 0 0" rpy="${m_pi} ${-m_pi_2} 0" /> -->
-      <origin xyz="0 0 0" rpy="0 0 0" />
-     <parent link="${prefix}link_6" />
-      <child link="${prefix}robotiq_85_adapter_link" />
-     <axis xyz="0 0 0"/> <!-- no rotation -->
-    </joint>
     <!-- ROS base_link to Fanuc World Coordinates transform -->
     <link name="${prefix}base" />
@@ -141,229 +134,4 @@
       <child link="${prefix}base"/>
     </joint>
-  <link name="${prefix}robotiq_85_adapter_link">
-    <visual>
-      <geometry>
-        <mesh filename="package://fanuc_lrmate200id_support/meshes/robotiq_c2/visual/robotiq_85_gripper_adapter_plate.dae"/>
-      </geometry>
-      <origin rpy="1.5707 0 1.5707" xyz="0 0 0"/>
-    </visual>
-    <collision>
-      <geometry>
-        <mesh filename="package://fanuc_lrmate200id_support/meshes/robotiq_c2/collision/robotiq_85_gripper_adapter_plate.dae"/>
-      </geometry>
-      <origin rpy="0 0 1.5707" xyz="0 0 0"/>
-    </collision>
-  </link>
-  <!--  /\  -->
-  <joint name="${prefix}robotiq_85_base_joint" type="fixed">
-    <parent link="${prefix}robotiq_85_adapter_link"/>
-    <child link="${prefix}robotiq_85_base_link"/>
-    <axis xyz="1 0 0"/>
-    <origin rpy="0 0 0" xyz=".0085 0 -.0041"/>
-  </joint>
-  <!--  \/  -->
-  <link name="${prefix}robotiq_85_base_link">
-    <visual>
-      <geometry>
-        <mesh filename="package://fanuc_lrmate200id_support/meshes/robotiq_c2/visual/robotiq_85_gripper_base.dae"/>
-      </geometry>
-      <origin rpy="3.1415 0 1.5707" xyz="0 0 0"/>
-    </visual>
-    <collision>
-      <geometry>
-        <mesh filename="package://fanuc_lrmate200id_support/meshes/robotiq_c2/collision/robotiq_85_gripper_base.dae"/>
-      </geometry>
-      <origin rpy="1.5707 0 1.5707" xyz="0 0 0"/>
-    </collision>
-  </link>
-  <!--  /\  -->
-  <!--  /\  -->
-  <joint name="${prefix}robotiq_85_left_knuckle_joint" type="revolute">
-    <parent link="${prefix}robotiq_85_base_link"/>
-    <child link="${prefix}robotiq_85_left_knuckle_link"/>
-    <axis xyz="1 0 0"/>
-    <origin rpy="-1.5707 1.5707 0" xyz=".04191 .0306 0"/>
-    <limit lower="0" upper=".8575" velocity="2.0" effort="1000"/>
-  </joint>
-  <joint name="${prefix}robotiq_85_right_knuckle_joint" type="revolute">
-    <parent link="${prefix}robotiq_85_base_link"/>
-    <child link="${prefix}robotiq_85_right_knuckle_link"/>
-    <axis xyz="1 0 0"/>
-    <origin rpy="1.5707 -1.5707 0" xyz=".04191 -.0306 0"/>
-    <limit lower="0" upper="1.5707" velocity="2.0" effort="1000"/>
-    <mimic joint="${prefix}robotiq_85_left_knuckle_joint" multiplier="1"/>
-  </joint>
-  <!--  \/  -->
-  <!--  \/  -->
-  <link name="${prefix}robotiq_85_left_knuckle_link">
-    <visual>
-      <geometry>
-        <mesh filename="package://fanuc_lrmate200id_support/meshes/robotiq_c2/visual/robotiq_85_gripper_joint_0_L.dae"/>
-      </geometry>
-      <origin rpy="3.14159 -1.5707 0" xyz="0 .04191 -.0306"/>
-    </visual>
-    <collision>
-      <geometry>
-        <mesh filename="package://fanuc_lrmate200id_support/meshes/robotiq_c2/collision/robotiq_85_gripper_joint_0_L.dae"/>
-      </geometry>
-      <origin rpy="1.5707 -1.5707 0" xyz="0 .04191 -.0306"/>
-    </collision>
-  </link>
-  <link name="${prefix}robotiq_85_right_knuckle_link">
-    <visual>
-      <geometry>
-        <mesh filename="package://fanuc_lrmate200id_support/meshes/robotiq_c2/visual/robotiq_85_gripper_joint_0_R.dae"/>
-      </geometry>
-      <origin rpy="3.14159 1.5707 0" xyz="0 .04191 -.0306"/>
-    </visual>
-    <collision>
-      <geometry>
-        <mesh filename="package://fanuc_lrmate200id_support/meshes/robotiq_c2/collision/robotiq_85_gripper_joint_0_R.dae"/>
-      </geometry>
-      <origin rpy="1.5707 1.5707 0" xyz="0 .04191 -.0306"/>
-    </collision>
-  </link>
-  <!--  /\  -->
-  <!--  /\  -->
-  <joint name="${prefix}robotiq_85_left_finger_joint" type="fixed">
-    <parent link="${prefix}robotiq_85_left_knuckle_link"/>
-    <child link="${prefix}robotiq_85_left_finger_link"/>
-    <axis xyz="1 0 0"/>
-    <origin rpy="3.1415 0 0" xyz="0 .00508 .03134"/>
-    <limit lower="0" upper="1.5707" velocity="2.0" effort="1000"/>
-  </joint>
-  <joint name="${prefix}robotiq_85_right_finger_joint" type="fixed">
-    <parent link="${prefix}robotiq_85_right_knuckle_link"/>
-    <child link="${prefix}robotiq_85_right_finger_link"/>
-    <axis xyz="1 0 0"/>
-    <origin rpy="3.1415 0 0" xyz="0 .00508 .03134"/>
-    <limit lower="0" upper="1.5707" velocity="2.0" effort="1000"/>
-  </joint>
-  <!--  \/  -->
-  <!--  \/  -->
-  <link name="${prefix}robotiq_85_left_finger_link">
-    <visual>
-      <geometry>
-        <mesh filename="package://fanuc_lrmate200id_support/meshes/robotiq_c2/visual/robotiq_85_gripper_joint_1_L.dae"/>
-      </geometry>
-      <origin rpy="0 1.5707 0" xyz="0 -.03683 .06194"/>
-    </visual>
-    <collision>
-      <geometry>
-        <mesh filename="package://fanuc_lrmate200id_support/meshes/robotiq_c2/collision/robotiq_85_gripper_joint_1_L.dae"/>
-      </geometry>
-      <origin rpy="-1.5707 1.5707 0" xyz="0 -.03683 .06194"/>
-    </collision>
-  </link>
-  <link name="${prefix}robotiq_85_right_finger_link">
-    <visual>
-      <geometry>
-        <mesh filename="package://fanuc_lrmate200id_support/meshes/robotiq_c2/visual/robotiq_85_gripper_joint_1_R.dae"/>
-      </geometry>
-      <origin rpy="0 -1.5707 0" xyz="0 -.03683 .06194"/>
-    </visual>
-    <collision>
-      <geometry>
-        <mesh filename="package://fanuc_lrmate200id_support/meshes/robotiq_c2/collision/robotiq_85_gripper_joint_1_R.dae"/>
-      </geometry>
-      <origin rpy="-1.5707 -1.5707 0" xyz="0 -.03683 .06194"/>
-    </collision>
-  </link>
-  <!--  /\  -->
-  <!--  /\  -->
-  <joint name="${prefix}robotiq_85_left_inner_knuckle_joint" type="revolute">
-    <parent link="${prefix}robotiq_85_base_link"/>
-    <child link="${prefix}robotiq_85_left_inner_knuckle_link"/>
-    <axis xyz="1 0 0"/>
-    <origin rpy="1.5707 1.5707 0" xyz=".04843 .0127 0"/>
-    <limit lower="0" upper="1.5707" velocity="2.0" effort="1000"/>
-    <mimic joint="${prefix}robotiq_85_left_knuckle_joint" offset="0"/>
-  </joint>
-  <joint name="${prefix}robotiq_85_right_inner_knuckle_joint" type="revolute">
-    <parent link="${prefix}robotiq_85_base_link"/>
-    <child link="${prefix}robotiq_85_right_inner_knuckle_link"/>
-    <axis xyz="1 0 0"/>
-    <origin rpy="-1.5707 -1.5707 0" xyz=".04843 -.0127 0"/>
-    <limit lower="0" upper="1.5707" velocity="2.0" effort="1000"/>
-    <mimic joint="${prefix}robotiq_85_left_knuckle_joint" offset="0"/>
-  </joint>
-  <!--  \/  -->
-  <!--  \/  -->
-  <link name="${prefix}robotiq_85_left_inner_knuckle_link">
-    <visual>
-      <geometry>
-        <mesh filename="package://fanuc_lrmate200id_support/meshes/robotiq_c2/visual/robotiq_85_gripper_joint_2_L.dae"/>
-      </geometry>
-      <origin rpy="0 1.5707 0" xyz="0 -.04843 .0127"/>
-    </visual>
-    <collision>
-      <geometry>
-        <mesh filename="package://fanuc_lrmate200id_support/meshes/robotiq_c2/collision/robotiq_85_gripper_joint_2_L.dae"/>
-      </geometry>
-      <origin rpy="-1.5707 1.5707 0" xyz="0 -.04843 .0127"/>
-    </collision>
-  </link>
-  <link name="${prefix}robotiq_85_right_inner_knuckle_link">
-    <visual>
-      <geometry>
-        <mesh filename="package://fanuc_lrmate200id_support/meshes/robotiq_c2/visual/robotiq_85_gripper_joint_2_R.dae"/>
-      </geometry>
-      <origin rpy="0 -1.5707 0" xyz="0 -.04843 .0127"/>
-    </visual>
-    <collision>
-      <geometry>
-        <mesh filename="package://fanuc_lrmate200id_support/meshes/robotiq_c2/collision/robotiq_85_gripper_joint_2_R.dae"/>
-      </geometry>
-      <origin rpy="-1.5707 -1.5707 0" xyz="0 -.04843 .0127"/>
-    </collision>
-  </link>
-  <!--  /\  -->
-  <!--  /\  -->
-  <joint name="${prefix}robotiq_85_left_finger_tip_joint" type="revolute">
-    <parent link="${prefix}robotiq_85_left_inner_knuckle_link"/>
-    <child link="${prefix}robotiq_85_left_finger_tip_link"/>
-    <axis xyz="1 0 0"/>
-    <origin rpy="0 0 0" xyz="0 .04196 -.0388"/>
-    <limit lower="0" upper="1.5707" velocity="2.0" effort="1000"/>
-    <mimic joint="${prefix}robotiq_85_left_knuckle_joint" multiplier="-1"/>
-  </joint>
-  <joint name="${prefix}robotiq_85_right_finger_tip_joint" type="revolute">
-    <parent link="${prefix}robotiq_85_right_inner_knuckle_link"/>
-    <child link="${prefix}robotiq_85_right_finger_tip_link"/>
-    <axis xyz="1 0 0"/>
-    <origin rpy="0 0 0" xyz="0 .04196 -.0388"/>
-    <limit lower="0" upper="1.5707" velocity="2.0" effort="1000"/>
-    <mimic joint="${prefix}robotiq_85_left_knuckle_joint" multiplier="-1"/>
-  </joint>
-  <!--  \/  -->
-  <!--  \/  -->
-  <link name="${prefix}robotiq_85_left_finger_tip_link">
-    <visual>
-      <geometry>
-        <mesh filename="package://fanuc_lrmate200id_support/meshes/robotiq_c2/visual/robotiq_85_gripper_joint_3_L.dae"/>
-      </geometry>
-      <origin rpy="0 1.5707 0" xyz="0 -.090381 .051505"/>
-    </visual>
-    <collision>
-      <geometry>
-        <mesh filename="package://fanuc_lrmate200id_support/meshes/robotiq_c2/collision/robotiq_85_gripper_joint_3_L.dae"/>
-      </geometry>
-      <origin rpy="-1.5707 1.5707 0" xyz="0 -.090381 .051505"/>
-    </collision>
-  </link>
-  <link name="${prefix}robotiq_85_right_finger_tip_link">
-    <visual>
-      <geometry>
-        <mesh filename="package://fanuc_lrmate200id_support/meshes/robotiq_c2/visual/robotiq_85_gripper_joint_3_R.dae"/>
-      </geometry>
-      <origin rpy="0 -1.5707 0" xyz="0 -.090381 .051505"/>
-    </visual>
-    <collision>
-      <geometry>
-        <mesh filename="package://fanuc_lrmate200id_support/meshes/robotiq_c2/collision/robotiq_85_gripper_joint_3_R.dae"/>
-      </geometry>
-      <origin rpy="-1.5707 -1.5707 0" xyz="0 -.090381 .051505"/>
-    </collision>
-  </link>
   </xacro:macro>
 </robot>
