Commit message: trac_ik motoman kin

File: nistfanuc_ws/src/robotduo/urdf/robotduo.xacro (robot description, xacro)
@@ -39,5 +39,5 @@
    <joint name="motoman_link_t-tool0" type="fixed" >
      <!--  <origin xyz="0 0 0.0" rpy="0 0 -3.1416"/> -->
-     <origin xyz="0 0 0.0" rpy="0  -1.57  0"/>
+     <origin xyz="0 0 0.0" rpy="0  0  -3.1416"/>
       <parent link="motoman_link_t" />
       <child link="motoman_robotiq_85_adapter_link" />
