Commit message: upgrade to kinetic broke stuff

File: nistcrcl_ws/src/fanuc_lrmate200id_support/urdf/lrmate200id_macro.xacro (robot description, xacro)
@@ -144,5 +144,5 @@
     <visual>
       <geometry>
-        <mesh filename="package://robotiq_c2_model_visualization/meshes/robotiq_c2/visual/robotiq_85_gripper_adapter_plate.dae"/>
+        <mesh filename="package://fanuc_lrmate200id_support/meshes/robotiq_c2/visual/robotiq_85_gripper_adapter_plate.dae"/>
       </geometry>
       <origin rpy="1.5707 0 1.5707" xyz="0 0 0"/>
@@ -150,5 +150,5 @@
     <collision>
       <geometry>
-        <mesh filename="package://robotiq_c2_model_visualization/meshes/robotiq_c2/collision/robotiq_85_gripper_adapter_plate.dae"/>
+        <mesh filename="package://fanuc_lrmate200id_support/meshes/robotiq_c2/collision/robotiq_85_gripper_adapter_plate.dae"/>
       </geometry>
       <origin rpy="0 0 1.5707" xyz="0 0 0"/>
@@ -166,5 +166,5 @@
     <visual>
       <geometry>
-        <mesh filename="package://robotiq_c2_model_visualization/meshes/robotiq_c2/visual/robotiq_85_gripper_base.dae"/>
+        <mesh filename="package://fanuc_lrmate200id_support/meshes/robotiq_c2/visual/robotiq_85_gripper_base.dae"/>
       </geometry>
       <origin rpy="3.1415 0 1.5707" xyz="0 0 0"/>
@@ -172,5 +172,5 @@
     <collision>
       <geometry>
-        <mesh filename="package://robotiq_c2_model_visualization/meshes/robotiq_c2/collision/robotiq_85_gripper_base.dae"/>
+        <mesh filename="package://fanuc_lrmate200id_support/meshes/robotiq_c2/collision/robotiq_85_gripper_base.dae"/>
       </geometry>
       <origin rpy="1.5707 0 1.5707" xyz="0 0 0"/>
@@ -199,5 +199,5 @@
     <visual>
       <geometry>
-        <mesh filename="package://robotiq_c2_model_visualization/meshes/robotiq_c2/visual/robotiq_85_gripper_joint_0_L.dae"/>
+        <mesh filename="package://fanuc_lrmate200id_support/meshes/robotiq_c2/visual/robotiq_85_gripper_joint_0_L.dae"/>
       </geometry>
       <origin rpy="3.14159 -1.5707 0" xyz="0 .04191 -.0306"/>
@@ -205,5 +205,5 @@
     <collision>
       <geometry>
-        <mesh filename="package://robotiq_c2_model_visualization/meshes/robotiq_c2/collision/robotiq_85_gripper_joint_0_L.dae"/>
+        <mesh filename="package://fanuc_lrmate200id_support/meshes/robotiq_c2/collision/robotiq_85_gripper_joint_0_L.dae"/>
       </geometry>
       <origin rpy="1.5707 -1.5707 0" xyz="0 .04191 -.0306"/>
@@ -213,5 +213,5 @@
     <visual>
       <geometry>
-        <mesh filename="package://robotiq_c2_model_visualization/meshes/robotiq_c2/visual/robotiq_85_gripper_joint_0_R.dae"/>
+        <mesh filename="package://fanuc_lrmate200id_support/meshes/robotiq_c2/visual/robotiq_85_gripper_joint_0_R.dae"/>
       </geometry>
       <origin rpy="3.14159 1.5707 0" xyz="0 .04191 -.0306"/>
@@ -219,5 +219,5 @@
     <collision>
       <geometry>
-        <mesh filename="package://robotiq_c2_model_visualization/meshes/robotiq_c2/collision/robotiq_85_gripper_joint_0_R.dae"/>
+        <mesh filename="package://fanuc_lrmate200id_support/meshes/robotiq_c2/collision/robotiq_85_gripper_joint_0_R.dae"/>
       </geometry>
       <origin rpy="1.5707 1.5707 0" xyz="0 .04191 -.0306"/>
@@ -245,5 +245,5 @@
     <visual>
       <geometry>
-        <mesh filename="package://robotiq_c2_model_visualization/meshes/robotiq_c2/visual/robotiq_85_gripper_joint_1_L.dae"/>
+        <mesh filename="package://fanuc_lrmate200id_support/meshes/robotiq_c2/visual/robotiq_85_gripper_joint_1_L.dae"/>
       </geometry>
       <origin rpy="0 1.5707 0" xyz="0 -.03683 .06194"/>
@@ -251,5 +251,5 @@
     <collision>
       <geometry>
-        <mesh filename="package://robotiq_c2_model_visualization/meshes/robotiq_c2/collision/robotiq_85_gripper_joint_1_L.dae"/>
+        <mesh filename="package://fanuc_lrmate200id_support/meshes/robotiq_c2/collision/robotiq_85_gripper_joint_1_L.dae"/>
       </geometry>
       <origin rpy="-1.5707 1.5707 0" xyz="0 -.03683 .06194"/>
@@ -259,5 +259,5 @@
     <visual>
       <geometry>
-        <mesh filename="package://robotiq_c2_model_visualization/meshes/robotiq_c2/visual/robotiq_85_gripper_joint_1_R.dae"/>
+        <mesh filename="package://fanuc_lrmate200id_support/meshes/robotiq_c2/visual/robotiq_85_gripper_joint_1_R.dae"/>
       </geometry>
       <origin rpy="0 -1.5707 0" xyz="0 -.03683 .06194"/>
@@ -265,5 +265,5 @@
     <collision>
       <geometry>
-        <mesh filename="package://robotiq_c2_model_visualization/meshes/robotiq_c2/collision/robotiq_85_gripper_joint_1_R.dae"/>
+        <mesh filename="package://fanuc_lrmate200id_support/meshes/robotiq_c2/collision/robotiq_85_gripper_joint_1_R.dae"/>
       </geometry>
       <origin rpy="-1.5707 -1.5707 0" xyz="0 -.03683 .06194"/>
@@ -293,5 +293,5 @@
     <visual>
       <geometry>
-        <mesh filename="package://robotiq_c2_model_visualization/meshes/robotiq_c2/visual/robotiq_85_gripper_joint_2_L.dae"/>
+        <mesh filename="package://fanuc_lrmate200id_support/meshes/robotiq_c2/visual/robotiq_85_gripper_joint_2_L.dae"/>
       </geometry>
       <origin rpy="0 1.5707 0" xyz="0 -.04843 .0127"/>
@@ -299,5 +299,5 @@
     <collision>
       <geometry>
-        <mesh filename="package://robotiq_c2_model_visualization/meshes/robotiq_c2/collision/robotiq_85_gripper_joint_2_L.dae"/>
+        <mesh filename="package://fanuc_lrmate200id_support/meshes/robotiq_c2/collision/robotiq_85_gripper_joint_2_L.dae"/>
       </geometry>
       <origin rpy="-1.5707 1.5707 0" xyz="0 -.04843 .0127"/>
@@ -307,5 +307,5 @@
     <visual>
       <geometry>
-        <mesh filename="package://robotiq_c2_model_visualization/meshes/robotiq_c2/visual/robotiq_85_gripper_joint_2_R.dae"/>
+        <mesh filename="package://fanuc_lrmate200id_support/meshes/robotiq_c2/visual/robotiq_85_gripper_joint_2_R.dae"/>
       </geometry>
       <origin rpy="0 -1.5707 0" xyz="0 -.04843 .0127"/>
@@ -313,5 +313,5 @@
     <collision>
       <geometry>
-        <mesh filename="package://robotiq_c2_model_visualization/meshes/robotiq_c2/collision/robotiq_85_gripper_joint_2_R.dae"/>
+        <mesh filename="package://fanuc_lrmate200id_support/meshes/robotiq_c2/collision/robotiq_85_gripper_joint_2_R.dae"/>
       </geometry>
       <origin rpy="-1.5707 -1.5707 0" xyz="0 -.04843 .0127"/>
@@ -341,5 +341,5 @@
     <visual>
       <geometry>
-        <mesh filename="package://robotiq_c2_model_visualization/meshes/robotiq_c2/visual/robotiq_85_gripper_joint_3_L.dae"/>
+        <mesh filename="package://fanuc_lrmate200id_support/meshes/robotiq_c2/visual/robotiq_85_gripper_joint_3_L.dae"/>
       </geometry>
       <origin rpy="0 1.5707 0" xyz="0 -.090381 .051505"/>
@@ -347,5 +347,5 @@
     <collision>
       <geometry>
-        <mesh filename="package://robotiq_c2_model_visualization/meshes/robotiq_c2/collision/robotiq_85_gripper_joint_3_L.dae"/>
+        <mesh filename="package://fanuc_lrmate200id_support/meshes/robotiq_c2/collision/robotiq_85_gripper_joint_3_L.dae"/>
       </geometry>
       <origin rpy="-1.5707 1.5707 0" xyz="0 -.090381 .051505"/>
@@ -355,5 +355,5 @@
     <visual>
       <geometry>
-        <mesh filename="package://robotiq_c2_model_visualization/meshes/robotiq_c2/visual/robotiq_85_gripper_joint_3_R.dae"/>
+        <mesh filename="package://fanuc_lrmate200id_support/meshes/robotiq_c2/visual/robotiq_85_gripper_joint_3_R.dae"/>
       </geometry>
       <origin rpy="0 -1.5707 0" xyz="0 -.090381 .051505"/>
@@ -361,5 +361,5 @@
     <collision>
       <geometry>
-        <mesh filename="package://robotiq_c2_model_visualization/meshes/robotiq_c2/collision/robotiq_85_gripper_joint_3_R.dae"/>
+        <mesh filename="package://fanuc_lrmate200id_support/meshes/robotiq_c2/collision/robotiq_85_gripper_joint_3_R.dae"/>
       </geometry>
       <origin rpy="-1.5707 -1.5707 0" xyz="0 -.090381 .051505"/>

File: nistfanuc_ws/src/fanuc_lrmate200id_support/urdf/lrmate200id_macro.xacro (robot description, xacro)
@@ -87,4 +87,5 @@
     <joint name="${prefix}joint_1" type="revolute">
       <origin xyz="0 0 0.330" rpy="0 0 0" />
+     <!-- <origin xyz="0 0 0.330" rpy="0 0 0" />-->
       <parent link="${prefix}base_link" />
       <child link="${prefix}link_1" />
@@ -130,5 +131,5 @@
     <link name="${prefix}base" />
     <joint name="${prefix}base_link-base" type="fixed">
-      <origin xyz="0 0 0.330" rpy="0 0 0"/>
+      <origin xyz="0 0 0" rpy="0 0 0"/>
       <parent link="${prefix}base_link"/>
       <child link="${prefix}base"/>
